Commit message: d

File: catkin_ws/src/multi_robot_scenario/xacro/laser/hokuyo.xacro (robot description, xacro)
@@ -2,5 +2,5 @@
 <robot xmlns:xacro="http://www.ros.org/wiki/xacro">
 <!-- Front Laser -->
-<xacro:macro name="laser" params="name parent xyz rpy meshes" >
+<xacro:macro name="laser" params="name parent xyz rpy meshes robotNamespace robot_name">
   <joint name="${parent}_${name}_joint" type="fixed">
       <axis xyz="0 0 1" />
@@ -48,5 +48,5 @@
           </ray>
           <plugin name="laser" filename="libgazebo_ros_laser.so" >
-            <robotNamespace></robotNamespace>
+            <robotNamespace>${robotNamespace}</robotNamespace>  <!-- abdel: Use argument -->
             <topicName>${name}/scan</topicName>
             <frameName>${name}</frameName>

File: catkin_ws/src/multi_robot_scenario/xacro/p3dx/pioneer3dx.xacro (robot description, xacro)
@@ -17,5 +17,7 @@
       xyz="0.125 0 0.25"
       rpy="0 0 0"
-      meshes="package://gazebo_plugins/test/multi_robot_scenario/meshes/laser"/>
+      meshes="package://gazebo_plugins/test/multi_robot_scenario/meshes/laser"
+      robotNamespace="/${robot_name}"
+      robot_name="${robot_name}" />
   <!-- ================= RGB Camera =================== -->
   <xacro:include filename="$(find multi_robot_scenario)/xacro/camera/camera.xacro"/>
